Commit message: pipeline

File: src/my_robot_description/urdf/arm.xacro (robot description, xacro)
@@ -123,12 +123,80 @@
     </collision>
   </link>
+  <link name="magician_link_gripper_core">
+    <inertial>
+      <mass value="0.05"/>
+      <origin xyz="0 0 0" rpy="0 0 0"/>
+      <inertia ixx="0.00001042" ixy="0.0" ixz="0.0"
+               iyy="0.00001417" iyz="0.0"
+               izz="0.00001667"/>
+    </inertial>
+    <visual>
+      <origin rpy="0 0 0" xyz="-8.06784046553505e-05 0 -0.027843407267811"/>
+      <geometry>
+        <mesh filename="package://my_robot_description/meshes/dae/gripper_core.dae"/>
+      </geometry>
+    </visual>
+    <collision>
+      <origin rpy="0 0 0" xyz="-8.06784046553505e-05 0 -0.027843407267811"/>
+      <geometry>
+        <mesh filename="package://my_robot_description/meshes/dae/gripper_core.dae"/>
+      </geometry>
+    </collision>
+  </link>
+  <link name="magician_link_gripper_jaw_left">
+    <inertial>
+      <mass value="0.01"/>
+      <origin xyz="0 0 0" rpy="0 0 0"/>
+      <inertia ixx="0.00000038" ixy="0.0" ixz="0.0"
+               iyy="0.00000108" iyz="0.0"
+               izz="0.00000080"/>
+    </inertial>
+    <visual>
+      <origin rpy="0 0 0" xyz="-8.06784046553505e-05 -0.0009 -0.027843407267811"/>
+      <geometry>
+        <mesh filename="package://my_robot_description/meshes/dae/jaw_left.dae"/>
+      </geometry>
+    </visual>
+    <collision>
+      <origin rpy="0 0 0" xyz="-8.06784046553505e-05 -0.0009 -0.027843407267811"/>
+      <geometry>
+        <mesh filename="package://my_robot_description/meshes/dae/jaw_left.dae"/>
+      </geometry>
+    </collision>
+  </link>
+  <link name="magician_link_gripper_jaw_right">
+    <inertial>
+      <mass value="0.01"/>
+      <origin xyz="0 0 0" rpy="0 0 0"/>
+      <inertia ixx="0.00000038" ixy="0.0" ixz="0.0"
+               iyy="0.00000108" iyz="0.0"
+               izz="0.00000080"/>
+    </inertial>
+    <visual>
+      <origin rpy="0 0 0" xyz="-8.06784046553505e-05 0.0009 -0.027843407267811"/>
+      <geometry>
+        <mesh filename="package://my_robot_description/meshes/dae/jaw_right.dae"/>
+      </geometry>
+    </visual>
+    <collision>
+      <origin rpy="0 0 0" xyz="-8.06784046553505e-05 0.0009 -0.027843407267811"/>
+      <geometry>
+        <mesh filename="package://my_robot_description/meshes/dae/jaw_right.dae"/>
+      </geometry>
+    </collision>
+  </link>
   <link name="end_effector">
     <inertial>
-      <mass value="0.01"/>
-      <origin xyz="0 0 0" rpy="0 0 0"/>
-      <inertia ixx="0.00001" ixy="0.0" ixz="0.0"
-               iyy="0.00001" iyz="0.0"
-               izz="0.00001"/>
-    </inertial>
+      <mass value="0.005"/> <origin xyz="0 0 0" rpy="0 0 0"/>
+      <inertia ixx="0.0000001" ixy="0.0" ixz="0.0"
+               iyy="0.0000001" iyz="0.0"
+               izz="0.0000001"/>
+    </inertial>
+    <collision>
+      <origin xyz="0 0 0" rpy="0 0 0"/>
+      <geometry>
+        <sphere radius="0.002"/>
+      </geometry>
+    </collision>
   </link>
   <!-- Joints -->
@@ -176,7 +244,7 @@
     <axis xyz="0 1 0"/>
     <limit effort="10.0"
-           lower="0.0"
-           upper="6.283185307179586"
-           velocity="5.585053606381855"/>
+          lower="-1.5708"
+          upper="0.0873"
+          velocity="5.585053606381855"/>
     <origin rpy="0 0 0" xyz="0.147 0 0"/>
     <dynamics damping="0.3" friction="0.1"/>
@@ -188,15 +256,42 @@
     <axis xyz="0 1 0"/>
     <limit effort="10.0"
-           lower="0.0"
-           upper="6.283185307179586"
-           velocity="5.585053606381855"/>
+          lower="-1.5708"
+          upper="0.2618"
+          velocity="5.585053606381855"/>
     <origin rpy="0 0 0" xyz="0 0 0"/>
     <dynamics damping="0.3" friction="0.1"/>
     <mimic joint="magician_joint_3" multiplier="-1" offset="0"/>
   </joint>
+  <joint name="magician_joint_4" type="revolute">
+    <parent link="magician_link_4"/>
+    <child link="magician_link_gripper_core"/>
+    <axis xyz="0 0 1"/>
+    <limit effort="10.0"
+          lower="-2.6179938779914944"
+          upper="2.6179938779914944"
+          velocity="5.585053606381855"/>
+    <origin rpy="0 0 0" xyz="0.06 0 0"/>
+    <dynamics damping="0.3" friction="0.1"/>
+  </joint>
+  <joint name="magician_joint_prismatic_l" type="prismatic">
+    <parent link="magician_link_gripper_core"/>
+    <child link="magician_link_gripper_jaw_left"/>
+    <axis xyz="0 1 0"/>
+    <limit effort="50.0" lower="0.0" upper="0.0135" velocity="1.0"/>
+    <origin rpy="0 0 0" xyz="0 0 0"/>
+    <dynamics damping="0.01" friction="0.01"/>
+  </joint>
+  <joint name="magician_joint_prismatic_r" type="prismatic">
+    <parent link="magician_link_gripper_core"/>
+    <child link="magician_link_gripper_jaw_right"/>
+    <axis xyz="0 -1 0"/>
+    <limit effort="50.0" lower="0.0" upper="0.0135" velocity="1.0"/>
+    <origin rpy="0 0 0" xyz="0 0 0"/>
+    <dynamics damping="0.01" friction="0.01"/>
+  </joint>
   <joint name="joint_end_effector" type="fixed">
-    <parent link="magician_link_4"/>
+    <parent link="magician_link_gripper_core"/>
     <child link="end_effector"/>
-    <origin rpy="0 0 0" xyz="0.06 0 0"/>
+    <origin rpy="0 0 0" xyz="0.065 0 0"/>
   </joint>
 </robot>

File: src/my_robot_description/urdf/arm_camera.xacro (robot description, xacro)
@@ -44,5 +44,5 @@
         <parent link="world"/>
         <child link="tower_camera"/>
-        <origin xyz="0.4 0.5 0" rpy="0 0 -2.0"/>
+        <origin xyz="0.6 0.7 0" rpy="0 0 -2.0"/>
     </joint>
     <joint name="tower_camera_to_camera" type="fixed">

File: src/my_robot_description/urdf/arm_control.xacro (robot description, xacro)
@@ -32,4 +32,25 @@
             <state_interface name="position" />
         </joint>
+        <joint name="magician_joint_4">
+            <command_interface name="position">
+            <param name="min">-2.6179938779914944</param>
+            <param name="max">2.6179938779914944</param>
+            </command_interface>
+            <state_interface name="position" />
+        </joint>
+        <joint name="magician_joint_prismatic_l">
+            <command_interface name="position">
+            <param name="min">0.0</param>
+            <param name="max">0.0135</param>
+            </command_interface>
+            <state_interface name="position" />
+        </joint>
+        <joint name="magician_joint_prismatic_r">
+            <command_interface name="position">
+                <param name="min">0.0</param>
+                <param name="max">0.0135</param>
+            </command_interface>
+            <state_interface name="position"/>
+        </joint>
     </ros2_control>
 </robot>

File: src/my_robot_description/urdf/arm_gazebo.xacro (robot description, xacro)
@@ -31,3 +31,15 @@
         </sensor>
     </gazebo>
+    <gazebo reference="magician_link_gripper_jaw_left">
+    <mu1>50.0</mu1>
+    <mu2>50.0</mu2>
+    <kp>1000000.0</kp>
+    <kd>1.0</kd>
+  </gazebo>
+  <gazebo reference="magician_link_gripper_jaw_right">
+    <mu1>50.0</mu1>
+    <mu2>50.0</mu2>
+    <kp>1000000.0</kp>
+    <kd>1.0</kd>
+  </gazebo>
 </robot>
